File: BB/BB.sch (KiCad schematic (older format))
At the start: 234 parts, among them SW0 SW_Push, U1 AT90USB1286-AU, Y0 16Mhz

Commit message: Half Switches in Place on PCB
Fixed issue on switch 62 2u
Parts:
- MX62: footprint MX_Alps_Hybrid:MX-1U -> MX_Alps_Hybrid:MX-2U
Changed lines of the file:
@@
 EESchema Schematic File Version 4
+LIBS:BB-cache
 EELAYER 29 0
 EELAYER END
@@
 F 0 "MX62" H 7721 5402 60  0000 C CNN
 F 1 "MX-2U" H 7721 5328 20  0000 C CNN
-F 2 "MX_Alps_Hybrid:MX-1U" H 7610 5160 60  0001 C CNN
+F 2 "MX_Alps_Hybrid:MX-2U" H 7610 5160 60  0001 C CNN
 F 3 "" H 7610 5160 60  0001 C CNN
 	1    7635 5185

Commit message: 5 Rows Done
Fixed 2u key footprint on key 38
Parts:
- MX38: footprint MX_Alps_Hybrid:MX-1U -> MX_Alps_Hybrid:MX-2U
Changed lines of the file:
@@
 F 0 "MX38" H 13256 4527 60  0000 C CNN
 F 1 "MX-2U" H 13256 4453 20  0000 C CNN
-F 2 "MX_Alps_Hybrid:MX-1U" H 13145 4285 60  0001 C CNN
+F 2 "MX_Alps_Hybrid:MX-2U" H 13145 4285 60  0001 C CNN
 F 3 "" H 13145 4285 60  0001 C CNN
 	1    13170 4310
