File: BB/BB.kicad_pcb (KiCad board)
At the start: 2 copper layers, 234 parts, among them SW0 SW_Push, U1 AT90USB1286-AU, Y0 16Mhz

Commit message: Half Switches in Place on PCB
Fixed issue on switch 62 2u
Parts:
- MX62: footprint MX_Alps_Hybrid:MX-1U -> MX_Alps_Hybrid:MX-2U
- moved C0 395.7 mm to (500.6, 216.9)
- moved C1 395.7 mm to (482.9, 216.9)
- moved C2 395.7 mm to (487.3, 216.9)
- moved C3 395.7 mm to (491.7, 216.9)
- moved C4 395.7 mm to (496.1, 216.9)
- moved C6 395.7 mm to (509.4, 216.9)
- moved F0 395.7 mm to (460.3, 217.0)
- moved R1 395.7 mm to (469.7, 216.9)
- moved R3 395.7 mm to (478.5, 216.9)
- moved C5 395.7 mm to (505.0, 216.9)
- moved D100 395.7 mm to (471.8, 213.7)
- moved D103 395.7 mm to (466.1, 213.7)
- moved D105 395.7 mm to (460.3, 213.7)
- moved D108 395.7 mm to (523.6, 213.7)
- moved D82 395.7 mm to (489.1, 213.7)
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
Commit message: 4 rows placed
Parts:
- moved MX23 385.0 mm to (62.4, 167.2)
- moved MX22 372.2 mm to (43.3, 167.2)
- moved MX21 359.8 mm to (24.3, 167.2)
- moved MX49 302.5 mm to (201.0, 186.3)
- moved MX24 293.3 mm to (81.4, 167.2)
- moved MX58 283.8 mm to (377.1, 186.3)
- moved MX54 251.4 mm to (296.2, 186.3)
- moved MX48 243.0 mm to (181.9, 186.3)
- moved MX53 231.2 mm to (277.2, 186.3)
- moved MX57 220.5 mm to (353.4, 186.3)
- moved MX46 217.9 mm to (143.8, 186.3)
- moved MX52 210.3 mm to (258.2, 186.3)
- moved MX51 182.1 mm to (239.1, 186.3)
- moved MX55 149.6 mm to (315.3, 186.3)
- moved MX47 142.9 mm to (162.9, 186.3)
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Changed lines of the file:
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@@
   )
   (module MX_Alps_Hybrid:MX-1U (layer F.Cu)
-    (at 328.800001 -24.369999)
+    (at 24.26 167.17)
     (fp_text reference MX21 (at 0 3.175) (layer Dwgs.User)
       (effects (font (size 1 1) (thickness 0.15)))
@@
   )
   (module MX_Alps_Hybrid:MX-1U (layer F.Cu)
-    (at 349.000001 -45.209999)
+    (at 43.32 167.17)
     (fp_text reference MX22 (at 0 3.175) (layer Dwgs.User)
       (effects (font (size 1 1) (thickness 0.15)))
@@
   )
   (module MX_Alps_Hybrid:MX-1U (layer F.Cu)
-    (at 369.200001 -65.409999)
+    (at 62.36 167.17)
     (fp_text reference MX23 (at 0 3.175) (layer Dwgs.User)
       (effects (font (size 1 1) (thickness 0.15)))
@@
   )
   (module MX_Alps_Hybrid:MX-1U (layer F.Cu)
-    (at 345.568001 39.840001)
+    (at 81.4 167.17)
     (fp_text reference MX24 (at 0 3.175) (layer Dwgs.User)
       (effects (font (size 1 1) (thickness 0.15)))
@@
   )
   (module MX_Alps_Hybrid:MX-1.5U (layer F.Cu)
-    (at 92.340501 61.960001)
+    (at 119.97 186.29)
     (fp_text reference MX45 (at 0 3.175) (layer Dwgs.User)
       (effects (font (size 1 1) (thickness 0.15)))
@@
   )
   (module MX_Alps_Hybrid:MX-1U (layer F.Cu)
-    (at 305.168001 39.840001)
+    (at 143.8 186.29)
     (fp_text reference MX46 (at 0 3.175) (layer Dwgs.User)
       (effects (font (size 1 1) (thickness 0.15)))
@@
   )
   (module MX_Alps_Hybrid:MX-1U (layer F.Cu)
-    (at 258.698001 80.240001)
+    (at 162.87 186.29)
     (fp_text reference MX47 (at 0 3.175) (layer Dwgs.User)
       (effects (font (size 1 1) (thickness 0.15)))
@@
   )
   (module MX_Alps_Hybrid:MX-1U (layer F.Cu)
-    (at 337.358001 -0.559999)
+    (at 181.93 186.29)
     (fp_text reference MX48 (at 0 3.175) (layer Dwgs.User)
       (effects (font (size 1 1) (thickness 0.15)))
@@
   )
   (module MX_Alps_Hybrid:MX-1U (layer F.Cu)
-    (at 333.560001 -85.609999)
+    (at 200.99 186.3)
     (fp_text reference MX49 (at 0 3.175) (layer Dwgs.User)
       (effects (font (size 1 1) (thickness 0.15)))
@@
   )
   (module MX_Alps_Hybrid:MX-1U (layer F.Cu)
-    (at 272.978001 60.040001)
+    (at 220.07 186.3)
     (fp_text reference MX50 (at 0 3.175) (layer Dwgs.User)
       (effects (font (size 1 1) (thickness 0.15)))
@@
   )
   (module MX_Alps_Hybrid:MX-1U (layer F.Cu)
-    (at 312.398001 19.640001)
+    (at 239.12 186.31)
     (fp_text reference MX51 (at 0 3.175) (layer Dwgs.User)
       (effects (font (size 1 1) (thickness 0.15)))
@@
   )
   (module MX_Alps_Hybrid:MX-1U (layer F.Cu)
-    (at 268.200001 -23.729999)
+    (at 258.16 186.31)
     (fp_text reference MX52 (at 0 3.175) (layer Dwgs.User)
       (effects (font (size 1 1) (thickness 0.15)))
@@
   )
   (module MX_Alps_Hybrid:MX-1U (layer F.Cu)
-    (at 288.400001 -44.569999)
+    (at 277.22 186.33)
     (fp_text reference MX53 (at 0 3.175) (layer Dwgs.User)
       (effects (font (size 1 1) (thickness 0.15)))
@@
   )
   (module MX_Alps_Hybrid:MX-1U (layer F.Cu)
-    (at 308.600001 -64.769999)
+    (at 296.25 186.35)
     (fp_text reference MX54 (at 0 3.175) (layer Dwgs.User)
       (effects (font (size 1 1) (thickness 0.15)))
@@
   )
   (module MX_Alps_Hybrid:MX-1U (layer F.Cu)
-    (at 284.968001 39.840001)
+    (at 315.28 186.34)
     (fp_text reference MX55 (at 0 3.175) (layer Dwgs.User)
       (effects (font (size 1 1) (thickness 0.15)))
@@
   )
   (module MX_Alps_Hybrid:MX-1U (layer F.Cu)
-    (at 238.498001 80.880001)
+    (at 334.32 186.34)
     (fp_text reference MX56 (at 0 3.175) (layer Dwgs.User)
       (effects (font (size 1 1) (thickness 0.15)))
@@
   )
   (module MX_Alps_Hybrid:MX-1U (layer F.Cu)
-    (at 288.400001 -24.369999)
+    (at 353.36 186.34)
     (fp_text reference MX57 (at 0 3.175) (layer Dwgs.User)
       (effects (font (size 1 1) (thickness 0.15)))
@@
   )
   (module MX_Alps_Hybrid:MX-1.5U (layer F.Cu)
-    (at 122.060501 61.960001)
+    (at 377.15 186.3)
     (fp_text reference MX58 (at 0 3.175) (layer Dwgs.User)
       (effects (font (size 1 1) (thickness 0.15)))

Commit message: 5 Rows Done
Fixed 2u key footprint on key 38
Parts:
- MX38: footprint MX_Alps_Hybrid:MX-1U -> MX_Alps_Hybrid:MX-2U
- moved MX31 291.7 mm to (229.5, 167.2)
- moved MX26 249.6 mm to (134.3, 167.2)
- moved MX34 240.8 mm to (286.7, 167.2)
- moved MX30 233.4 mm to (210.5, 167.2)
- moved MX35 213.0 mm to (305.7, 167.2)
- moved MX29 211.8 mm to (191.4, 167.2)
- moved MX25 203.4 mm to (115.2, 167.2)
- moved MX36 192.3 mm to (324.8, 167.2)
- moved MX28 191.6 mm to (172.4, 167.2)
- moved MX33 170.4 mm to (267.6, 167.2)
- moved MX27 163.2 mm to (153.3, 167.2)
- moved MX37 128.7 mm to (343.8, 167.2)
- moved MX38 127.7 mm to (372.4, 167.2)
- moved MX32 125.2 mm to (248.6, 167.2)
Changed lines of the file:
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@@
   )
   (module MX_Alps_Hybrid:MX-2U (layer F.Cu)
+    (at 372.38 167.22)
+    (fp_text reference MX38 (at 0 3.175) (layer Dwgs.User)
+      (effects (font (size 1 1) (thickness 0.15)))
+    )
+    (fp_text value MX-2U (at 0 -7.9375) (layer Dwgs.User)
+      (effects (font (size 1 1) (thickness 0.15)))
+    )
+    (fp_line (start -19.05 9.525) (end -19.05 -9.525) (layer Dwgs.User) (width 0.15))
+    (fp_line (start -19.05 9.525) (end 19.05 9.525) (layer Dwgs.User) (width 0.15))
+    (fp_line (start 19.05 -9.525) (end 19.05 9.525) (layer Dwgs.User) (width 0.15))
+    (fp_line (start -19.05 -9.525) (end 19.05 -9.525) (layer Dwgs.User) (width 0.15))
+    (fp_line (start -7 -7) (end -7 -5) (layer Dwgs.User) (width 0.15))
+    (fp_line (start -5 -7) (end -7 -7) (layer Dwgs.User) (width 0.15))
+    (fp_line (start -7 7) (end -5 7) (layer Dwgs.User) (width 0.15))
+    (fp_line (start -7 5) (end -7 7) (layer Dwgs.User) (width 0.15))
+    (fp_line (start 7 7) (end 7 5) (layer Dwgs.User) (width 0.15))
+    (fp_line (start 5 7) (end 7 7) (layer Dwgs.User) (width 0.15))
+    (fp_line (start 7 -7) (end 7 -5) (layer Dwgs.User) (width 0.15))
+    (fp_line (start 5 -7) (end 7 -7) (layer Dwgs.User) (width 0.15))
+    (pad "" np_thru_hole circle (at 11.938 8.255) (size 3.9878 3.9878) (drill 3.9878) (layers *.Cu *.Mask))
+    (pad "" np_thru_hole circle (at -11.938 8.255) (size 3.9878 3.9878) (drill 3.9878) (layers *.Cu *.Mask))
+    (pad "" np_thru_hole circle (at 11.938 -6.985) (size 3.048 3.048) (drill 3.048) (layers *.Cu *.Mask))
+    (pad "" np_thru_hole circle (at -11.938 -6.985) (size 3.048 3.048) (drill 3.048) (layers *.Cu *.Mask))
+    (pad "" np_thru_hole circle (at 5.08 0 48.0996) (size 1.75 1.75) (drill 1.75) (layers *.Cu *.Mask))
+    (pad "" np_thru_hole circle (at -5.08 0 48.0996) (size 1.75 1.75) (drill 1.75) (layers *.Cu *.Mask))
+    (pad 4 thru_hole rect (at 1.27 5.08) (size 1.905 1.905) (drill 1.04) (layers *.Cu B.Mask)
+      (net 220 "Net-(MX38-Pad4)"))
+    (pad 3 thru_hole circle (at -1.27 5.08) (size 1.905 1.905) (drill 1.04) (layers *.Cu B.Mask)
+      (net 219 "Net-(MX38-Pad3)"))
+    (pad 1 thru_hole circle (at -2.5 -4) (size 2.25 2.25) (drill 1.47) (layers *.Cu B.Mask)
+      (net 173 COL18))
+    (pad "" np_thru_hole circle (at 0 0) (size 3.9878 3.9878) (drill 3.9878) (layers *.Cu *.Mask))
+    (pad 1 thru_hole oval (at -3.81 -2.54 48.0996) (size 4.211556 2.25) (drill 1.47 (offset 0.980778 0)) (layers *.Cu B.Mask)
+      (net 173 COL18))
+    (pad 2 thru_hole circle (at 2.54 -5.08) (size 2.25 2.25) (drill 1.47) (layers *.Cu B.Mask)
+      (net 45 "Net-(D38-Pad2)"))
+    (pad 2 thru_hole oval (at 2.5 -4.5 86.0548) (size 2.831378 2.25) (drill 1.47 (offset 0.290689 0)) (layers *.Cu B.Mask)
+      (net 45 "Net-(D38-Pad2)"))
+  )
+  (module MX_Alps_Hybrid:MX-2U (layer F.Cu)
     (at 81.41 195.76 270)
     (fp_text reference MX62 (at 0 3.175 270) (layer Dwgs.User)
@@
   )
   (module MX_Alps_Hybrid:MX-1U (layer F.Cu)
-    (at 299.098001 80.240001)
+    (at 115.21 167.25)
     (fp_text reference MX25 (at 0 3.175) (layer Dwgs.User)
       (effects (font (size 1 1) (thickness 0.15)))
@@
   )
   (module MX_Alps_Hybrid:MX-1U (layer F.Cu)
-    (at 227.800001 -64.129999)
+    (at 134.26 167.25)
     (fp_text reference MX26 (at 0 3.175) (layer Dwgs.User)
       (effects (font (size 1 1) (thickness 0.15)))
@@
   )
   (module MX_Alps_Hybrid:MX-1U (layer F.Cu)
-    (at 224.368001 20.280001)
+    (at 153.3 167.24)
     (fp_text reference MX27 (at 0 3.175) (layer Dwgs.User)
       (effects (font (size 1 1) (thickness 0.15)))
@@
   )
   (module MX_Alps_Hybrid:MX-1U (layer F.Cu)
-    (at 187.400001 -23.729999)
+    (at 172.36 167.24)
     (fp_text reference MX28 (at 0 3.175) (layer Dwgs.User)
       (effects (font (size 1 1) (thickness 0.15)))
@@
   )
   (module MX_Alps_Hybrid:MX-1U (layer F.Cu)
-    (at 207.600001 -43.929999)
+    (at 191.41 167.23)
     (fp_text reference MX29 (at 0 3.175) (layer Dwgs.User)
       (effects (font (size 1 1) (thickness 0.15)))
@@
   )
   (module MX_Alps_Hybrid:MX-1U (layer F.Cu)
-    (at 308.600001 -44.569999)
+    (at 210.48 167.22)
     (fp_text reference MX30 (at 0 3.175) (layer Dwgs.User)
       (effects (font (size 1 1) (thickness 0.15)))
@@
   )
   (module MX_Alps_Hybrid:MX-1U (layer F.Cu)
-    (at 373.960001 -86.249999)
+    (at 229.54 167.21)
     (fp_text reference MX31 (at 0 3.175) (layer Dwgs.User)
       (effects (font (size 1 1) (thickness 0.15)))
@@
   )
   (module MX_Alps_Hybrid:MX-1U (layer F.Cu)
-    (at 313.378001 60.040001)
+    (at 248.58 167.21)
     (fp_text reference MX32 (at 0 3.175) (layer Dwgs.User)
       (effects (font (size 1 1) (thickness 0.15)))
@@
   )
   (module MX_Alps_Hybrid:MX-1U (layer F.Cu)
-    (at 352.798001 19.640001)
+    (at 267.63 167.21)
     (fp_text reference MX33 (at 0 3.175) (layer Dwgs.User)
       (effects (font (size 1 1) (thickness 0.15)))
@@
   )
   (module MX_Alps_Hybrid:MX-1U (layer F.Cu)
-    (at 349.000001 -65.409999)
+    (at 286.68 167.21)
     (fp_text reference MX34 (at 0 3.175) (layer Dwgs.User)
       (effects (font (size 1 1) (thickness 0.15)))
@@
   )
   (module MX_Alps_Hybrid:MX-1U (layer F.Cu)
-    (at 328.800001 -44.569999)
+    (at 305.72 167.21)
     (fp_text reference MX35 (at 0 3.175) (layer Dwgs.User)
       (effects (font (size 1 1) (thickness 0.15)))
@@
   )
   (module MX_Alps_Hybrid:MX-1U (layer F.Cu)
-    (at 308.600001 -24.369999)
+    (at 324.75 167.21)
     (fp_text reference MX36 (at 0 3.175) (layer Dwgs.User)
       (effects (font (size 1 1) (thickness 0.15)))
@@
   )
   (module MX_Alps_Hybrid:MX-1U (layer F.Cu)
-    (at 325.368001 39.840001)
+    (at 343.81 167.22)
     (fp_text reference MX37 (at 0 3.175) (layer Dwgs.User)
       (effects (font (size 1 1) (thickness 0.15)))
@@
   )
   (module MX_Alps_Hybrid:MX-1U (layer F.Cu)
-    (at 278.898001 80.240001)
-    (fp_text reference MX38 (at 0 3.175) (layer Dwgs.User)
-      (effects (font (size 1 1) (thickness 0.15)))
-    )
-    (fp_text value MX-2U (at 0 -7.9375) (layer Dwgs.User)
-      (effects (font (size 1 1) (thickness 0.15)))
-    )
-    (fp_line (start 5 -7) (end 7 -7) (layer Dwgs.User) (width 0.15))
-    (fp_line (start 7 -7) (end 7 -5) (layer Dwgs.User) (width 0.15))
-    (fp_line (start 5 7) (end 7 7) (layer Dwgs.User) (width 0.15))
-    (fp_line (start 7 7) (end 7 5) (layer Dwgs.User) (width 0.15))
-    (fp_line (start -7 5) (end -7 7) (layer Dwgs.User) (width 0.15))
-    (fp_line (start -7 7) (end -5 7) (layer Dwgs.User) (width 0.15))
-    (fp_line (start -5 -7) (end -7 -7) (layer Dwgs.User) (width 0.15))
-    (fp_line (start -7 -7) (end -7 -5) (layer Dwgs.User) (width 0.15))
-    (fp_line (start -9.525 -9.525) (end 9.525 -9.525) (layer Dwgs.User) (width 0.15))
-    (fp_line (start 9.525 -9.525) (end 9.525 9.525) (layer Dwgs.User) (width 0.15))
-    (fp_line (start 9.525 9.525) (end -9.525 9.525) (layer Dwgs.User) (width 0.15))
-    (fp_line (start -9.525 9.525) (end -9.525 -9.525) (layer Dwgs.User) (width 0.15))
-    (pad 2 thru_hole oval (at 2.5 -4.5 86.0548) (size 2.831378 2.25) (drill 1.47 (offset 0.290689 0)) (layers *.Cu B.Mask)
-      (net 45 "Net-(D38-Pad2)"))
-    (pad 2 thru_hole circle (at 2.54 -5.08) (size 2.25 2.25) (drill 1.47) (layers *.Cu B.Mask)
-      (net 45 "Net-(D38-Pad2)"))
-    (pad 1 thru_hole oval (at -3.81 -2.54 48.0996) (size 4.211556 2.25) (drill 1.47 (offset 0.980778 0)) (layers *.Cu B.Mask)
-      (net 173 COL18))
-    (pad "" np_thru_hole circle (at 0 0) (size 3.9878 3.9878) (drill 3.9878) (layers *.Cu *.Mask))
-    (pad 1 thru_hole circle (at -2.5 -4) (size 2.25 2.25) (drill 1.47) (layers *.Cu B.Mask)
-      (net 173 COL18))
-    (pad 3 thru_hole circle (at -1.27 5.08) (size 1.905 1.905) (drill 1.04) (layers *.Cu B.Mask)
-      (net 219 "Net-(MX38-Pad3)"))
-    (pad 4 thru_hole rect (at 1.27 5.08) (size 1.905 1.905) (drill 1.04) (layers *.Cu B.Mask)
-      (net 220 "Net-(MX38-Pad4)"))
-    (pad "" np_thru_hole circle (at -5.08 0 48.0996) (size 1.75 1.75) (drill 1.75) (layers *.Cu *.Mask))
-    (pad "" np_thru_hole circle (at 5.08 0 48.0996) (size 1.75 1.75) (drill 1.75) (layers *.Cu *.Mask))
-  )
-  (module MX_Alps_Hybrid:MX-1U (layer F.Cu)

Commit message: Rows Done
Excluding Right Pad
Parts:
- moved MX8 393.5 mm to (90.3, 136.9)
- moved MX5 373.0 mm to (33.1, 136.9)
- moved MX6 347.6 mm to (52.2, 136.9)
- moved MX4 284.3 mm to (210.4, 136.9)
- moved MX7 274.2 mm to (71.2, 136.9)
- moved MX3 269.4 mm to (191.4, 136.9)
- moved MX9 250.6 mm to (115.2, 136.8)
- moved MX16 234.4 mm to (362.9, 136.9)
- moved MX13 223.3 mm to (296.2, 136.9)
- moved MX2 215.8 mm to (172.3, 136.8)
- moved MX10 193.7 mm to (239.0, 136.9)
- moved MX14 187.5 mm to (324.7, 136.9)
- moved MX11 185.7 mm to (258.1, 136.9)
- moved MX12 170.4 mm to (277.1, 136.9)
- moved MX1 169.5 mm to (153.3, 136.8)
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
Commit message: All Switches Placed
Diodes on Side
Parts:
- moved MX105 407.0 mm to (486.7, 211.6)
- moved USB0 364.0 mm to (195.7, 97.2), turned to 270 degrees
- moved MX85 328.3 mm to (505.8, 192.6)
- moved MX83 313.6 mm to (467.7, 192.5)
- moved MX61 307.0 mm to (505.8, 143.1)
- moved MX66 278.0 mm to (486.7, 173.5)
- moved MX84 260.3 mm to (486.7, 192.6)
- moved MX40 248.3 mm to (486.7, 124.1)
- moved MX41 222.0 mm to (505.7, 124.1)
- moved MX18 204.9 mm to (467.6, 105.0)
- moved D1 190.2 mm to (572.8, 39.9)
- moved D109 190.2 mm to (555.6, 39.9)
- moved D17 190.2 mm to (567.7, 36.6)
- moved D19 190.2 mm to (498.1, 40.6)
- moved D21 190.2 mm to (492.3, 40.6)
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
Commit message: All Componenets in Place on PCB
No routing, temporary MCU placement
Parts:
- moved D5 527.5 mm to (54.7, 85.5), turned to 90 degrees
- moved D6 516.9 mm to (73.8, 85.6), turned to 90 degrees
- moved D42 514.9 mm to (54.7, 134.9), turned to 90 degrees
- moved D64 506.1 mm to (73.8, 154.1), turned to 90 degrees
- moved D63 496.6 mm to (54.8, 154.1), turned to 90 degrees
- moved D43 494.0 mm to (73.8, 134.9), turned to 90 degrees
- moved D7 489.9 mm to (92.8, 85.6), turned to 90 degrees
- moved D80 479.3 mm to (54.7, 173.2), turned to 90 degrees
- moved D44 478.7 mm to (92.8, 138.1), turned to 90 degrees
- moved D23 478.1 mm to (92.8, 115.9), turned to 90 degrees
- moved D8 476.1 mm to (112.0, 85.5), turned to 90 degrees
- moved D24 467.5 mm to (111.9, 115.8), turned to 90 degrees
- moved D81 456.5 mm to (73.8, 173.2), turned to 90 degrees
- moved D62 451.5 mm to (103.5, 132.7)
- moved D100 450.7 mm to (72.2, 192.3), turned to 90 degrees
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
Commit message: Checkpoint Before Routing
Calm before the storm
Parts:
- moved C2 53.4 mm to (433.8, 137.9)
- moved C4 53.4 mm to (442.6, 137.9)
- moved C1 53.4 mm to (429.4, 137.9)
- moved C3 53.4 mm to (438.2, 137.9)
- moved R1 7.02 mm to (147.0, 86.0)
- moved F0 7.02 mm to (149.5, 80.5)
- moved R2 7.02 mm to (143.7, 86.1)
- moved USB0 7.02 mm to (146.3, 70.7)
Changed lines of the file:
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@@
   (general
     (thickness 1.6)
-    (drawings 0)
+    (drawings 8)
     (tracks 0)
     (zones 0)
@@
     (solder_mask_min_width 0.25)
     (aux_axis_origin 0 0)
-    (visible_elements 7FFFF7FF)
+    (visible_elements 7FFFFFFF)
     (pcbplotparams
       (layerselection 0x010fc_ffffffff)
@@
   )
   (module Capacitor_SMD:C_0805_2012Metric (layer F.Cu)
-    (at 409.737001 187.514001)
+    (at 429.407001 137.884001)
     (descr "Capacitor SMD 0805 (2012 Metric), square (rectangular) end terminal, IPC_7351 nominal, (Body size source: https://docs.google.com/spreadsheets/d/1BsfQQcO9C6DZCsRaXUlFlo91Tg2WpOkGARC1WS5S8t0/edit?usp=sharing), generated with kicad-footprint-generator")
     (tags capacitor)
@@
   )
   (module Capacitor_SMD:C_0805_2012Metric (layer F.Cu)
-    (at 414.147001 187.514001)
+    (at 433.817001 137.884001)
     (descr "Capacitor SMD 0805 (2012 Metric), square (rectangular) end terminal, IPC_7351 nominal, (Body size source: https://docs.google.com/spreadsheets/d/1BsfQQcO9C6DZCsRaXUlFlo91Tg2WpOkGARC1WS5S8t0/edit?usp=sharing), generated with kicad-footprint-generator")
     (tags capacitor)
@@
   )
   (module Capacitor_SMD:C_0805_2012Metric (layer F.Cu)
-    (at 418.557001 187.514001)
+    (at 438.227001 137.884001)
     (descr "Capacitor SMD 0805 (2012 Metric), square (rectangular) end terminal, IPC_7351 nominal, (Body size source: https://docs.google.com/spreadsheets/d/1BsfQQcO9C6DZCsRaXUlFlo91Tg2WpOkGARC1WS5S8t0/edit?usp=sharing), generated with kicad-footprint-generator")
     (tags capacitor)
@@
   )
   (module Capacitor_SMD:C_0805_2012Metric (layer F.Cu)
-    (at 422.967001 187.514001)
+    (at 442.637001 137.884001)
     (descr "Capacitor SMD 0805 (2012 Metric), square (rectangular) end terminal, IPC_7351 nominal, (Body size source: https://docs.google.com/spreadsheets/d/1BsfQQcO9C6DZCsRaXUlFlo91Tg2WpOkGARC1WS5S8t0/edit?usp=sharing), generated with kicad-footprint-generator")
     (tags capacitor)
@@
   )
   (module Fuse:Fuse_1206_3216Metric (layer F.Cu)
-    (at 149.54 87.49 90)
+    (at 149.51 80.47 90)
     (descr "Fuse SMD 1206 (3216 Metric), square (rectangular) end terminal, IPC_7351 nominal, (Body size source: http://www.tortai-tech.com/upload/download/2011102023233369053.pdf), generated with kicad-footprint-generator")
     (tags resistor)
@@
   )
   (module Resistor_SMD:R_0805_2012Metric (layer F.Cu)
-    (at 147.03 93.0275 90)
+    (at 147 86.0075 90)
     (descr "Resistor SMD 0805 (2012 Metric), square (rectangular) end terminal, IPC_7351 nominal, (Body size source: https://docs.google.com/spreadsheets/d/1BsfQQcO9C6DZCsRaXUlFlo91Tg2WpOkGARC1WS5S8t0/edit?usp=sharing), generated with kicad-footprint-generator")
     (tags resistor)
@@
   )
   (module Resistor_SMD:R_0805_2012Metric (layer F.Cu)
-    (at 143.68 93.0775 90)
+    (at 143.65 86.0575 90)
     (descr "Resistor SMD 0805 (2012 Metric), square (rectangular) end terminal, IPC_7351 nominal, (Body size source: https://docs.google.com/spreadsheets/d/1BsfQQcO9C6DZCsRaXUlFlo91Tg2WpOkGARC1WS5S8t0/edit?usp=sharing), generated with kicad-footprint-generator")
     (tags resistor)
@@
   )
   (module random-keyboard-parts:Molex-0548190589 (layer F.Cu)
-    (at 146.29 77.69 270)
+    (at 146.26 70.67 270)
     (attr smd)
     (fp_text reference USB0 (at 2.032 0) (layer F.SilkS)
@@
     )
   )
+  (gr_line (start 28.710543 74.628422) (end 28.64 203.11) (layer F.SilkS) (width 0.12))
+  (gr_line (start 473.22 74.49) (end 473.149457 202.971578) (layer F.SilkS) (width 0.12))
+  (gr_line (start 34.378422 208.769457) (end 467.49 208.71) (layer F.SilkS) (width 0.12))
+  (gr_arc (start 467.49 203.05) (end 467.49 208.71) (angle -90.79388609) (layer F.SilkS) (width 0.12))
+  (gr_arc (start 34.3 203.11) (end 28.64 203.11) (angle -90.79388609) (layer F.SilkS) (width 0.12))
+  (gr_line (start 467.481578 68.830543) (end 34.37 68.89) (layer F.SilkS) (width 0.12))
+  (gr_arc (start 34.37 74.55) (end 34.37 68.89) (angle -90.79388609) (layer F.SilkS) (width 0.12))
+  (gr_arc (start 467.56 74.49) (end 473.22 74.49) (angle -90.79388609) (layer F.SilkS) (width 0.12))
 )
