File: BB/BB.kicad_pcb (KiCad board)
At the start: 2 copper layers, 234 parts, among them SW0 SW_Push, U1 AT90USB1286-AU, Y0 16Mhz

Commit message: Rows Done
Main Columns
Parts:
- moved C0 79.5 mm to (484.1, 141.5)
- moved C5 72.8 mm to (484.4, 153.3)
- moved C6 72.8 mm to (492.3, 153.3)
- moved Y0 72.8 mm to (488.3, 153.2)
- moved R3 59.7 mm to (509.6, 129.5)
- moved C1 59.7 mm to (488.5, 129.7)
- moved C2 59.7 mm to (492.9, 129.7)
- moved C3 59.7 mm to (497.3, 129.7)
- moved C4 59.7 mm to (501.7, 129.7)
- moved R0 59.7 mm to (486.0, 134.2)
- moved SW0 46.5 mm to (501.0, 143.1)
- moved USB0 0.07 mm to (146.3, 70.6)
- turned U1 to 180 degrees
Connections:
- MX67 pad 3: COL4 -> Net-(MX67-Pad3)
- MX89 pad 1: Net-(MX89-Pad1) -> COL9
- U1 pad 25: Net-(U1-Pad25) -> ROW0
- U1 pad 26: Net-(U1-Pad26) -> ROW1
- U1 pad 27: Net-(U1-Pad27) -> ROW2
- U1 pad 28: Net-(U1-Pad28) -> ROW3
- U1 pad 29: Net-(U1-Pad29) -> ROW4
- U1 pad 30: Net-(U1-Pad30) -> ROW5
- U1 pad 31: Net-(U1-Pad31) -> ROW6
- U1 pad 37: Net-(U1-Pad37) -> COL0
- U1 pad 38: Net-(U1-Pad38) -> COL1
- U1 pad 39: Net-(U1-Pad39) -> COL2
- U1 pad 40: Net-(U1-Pad40) -> COL3
- U1 pad 41: Net-(U1-Pad41) -> COL4
- U1 pad 42: Net-(U1-Pad42) -> COL5
- U1 pad 44: Net-(U1-Pad44) -> COL6
- U1 pad 45: Net-(U1-Pad45) -> COL7
- U1 pad 46: Net-(U1-Pad46) -> COL8
- U1 pad 47: Net-(U1-Pad47) -> COL9
- U1 pad 48: Net-(U1-Pad48) -> COL10
- U1 pad 49: Net-(U1-Pad49) -> COL11
- U1 pad 50: Net-(U1-Pad50) -> COL12
- U1 pad 51: Net-(U1-Pad51) -> COL13
- U1 pad 54: Net-(U1-Pad54) -> COL14
- U1 pad 55: Net-(U1-Pad55) -> COL15
- U1 pad 56: Net-(U1-Pad56) -> COL16
- U1 pad 57: Net-(U1-Pad57) -> COL17
- U1 pad 58: Net-(U1-Pad58) -> COL18
- U1 pad 59: Net-(U1-Pad59) -> COL19
- U1 pad 60: Net-(U1-Pad60) -> COL20
- U1 pad 61: Net-(U1-Pad61) -> COL21
Routing:
- net COL14: track 0.00 -> 112.3 mm
- net COL2: track 0.00 -> 110.4 mm
- net COL1: track 0.00 -> 105.3 mm
- net COL7: track 0.00 -> 105.0 mm
- net COL11: track 0.00 -> 102.1 mm
- net COL16: track 0.00 -> 102.0 mm
- net COL17: track 0.00 -> 101.3 mm
- net COL18: track 0.00 -> 99.9 mm
- net COL6: track 0.00 -> 99.7 mm
- net COL4: track 0.00 -> 92.2 mm
- net COL3: track 0.00 -> 88.4 mm
- net COL0: track 0.00 -> 84.7 mm
- net COL5: track 0.00 -> 82.8 mm
- net COL13: track 0.00 -> 81.9 mm
- net COL9: track 0.00 -> 81.8 mm
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Other:
- net class Default: trace_width 0.25 -> 0.254
- net class Power added: clearance 0.2, trace_width 0.381, via_dia 0.8, via_drill 0.4
